Commit message: Feature:add the base_driver function and update the README,add some parameter of the base

File: src/spore_patrol_description/urdf/spore_patrol_robot.urdf.xacro (robot description, xacro)
@@ -2,15 +2,16 @@
 <robot xmlns:xacro="http://www.ros.org/wiki/xacro" name="spore_patrol_robot">
   <!--
-    Provisional geometry from the STM32 firmware's TOP_4WD_BS variant.
-    Replace these values after measuring the actual chassis and payload.
+    WHEELTEC high-configuration pendulum-suspension chassis.
+    Dimensions are from docs/小车相关参数/小车二维模型图纸.jpg.
+    The payload and sensor mounting positions remain provisional.
   -->
-  <xacro:property name="half_track" value="0.311"/>
-  <xacro:property name="half_wheelbase" value="0.308"/>
-  <xacro:property name="wheel_radius" value="0.1125"/>
-  <xacro:property name="wheel_width" value="0.085"/>
-  <xacro:property name="chassis_length" value="0.72"/>
-  <xacro:property name="chassis_width" value="0.56"/>
-  <xacro:property name="chassis_height" value="0.12"/>
-  <xacro:property name="chassis_z" value="0.19"/>
+  <xacro:property name="half_track" value="0.1678"/>
+  <xacro:property name="half_wheelbase" value="0.15635"/>
+  <xacro:property name="wheel_radius" value="0.076"/>
+  <xacro:property name="wheel_width" value="0.048"/>
+  <xacro:property name="chassis_length" value="0.3127"/>
+  <xacro:property name="chassis_width" value="0.238"/>
+  <xacro:property name="chassis_height" value="0.09"/>
+  <xacro:property name="chassis_z" value="0.096"/>
   <material name="orange">
     <color rgba="0.96 0.45 0.08 1.0"/>
@@ -37,6 +38,6 @@
     <inertial>
       <origin xyz="0 0 0"/>
-      <mass value="35.0"/>
-      <inertia ixx="1.25" ixy="0" ixz="0" iyy="1.65" iyz="0" izz="2.30"/>
+      <mass value="7.6"/>
+      <inertia ixx="0.12" ixy="0" ixz="0" iyy="0.17" iyz="0" izz="0.23"/>
     </inertial>
     <visual>
@@ -52,4 +53,10 @@
     </collision>
   </link>
+  <joint name="imu_joint" type="fixed">
+    <parent link="base_link"/>
+    <child link="imu_link"/>
+    <origin xyz="0 0 0" rpy="0 0 0"/>
+  </joint>
+  <link name="imu_link"/>
   <xacro:macro name="fixed_wheel" params="name x y">
     <joint name="${name}_joint" type="fixed">
@@ -81,10 +88,10 @@
     <parent link="base_link"/>
     <child link="sensor_deck"/>
-    <origin xyz="0 0 0.15"/>
+    <origin xyz="0 0 0.12"/>
   </joint>
   <link name="sensor_deck">
     <visual>
       <geometry>
-        <box size="0.58 0.44 0.045"/>
+        <box size="0.34 0.22 0.025"/>
       </geometry>
       <material name="silver"/>

Commit message: feat:增加了激光雷达的功能包，根据厂家的URDF文件完善了RViz模型，添加统一 实车启动入口，编写室内二维建图操作包

File: src/spore_patrol_description/urdf/spore_patrol_robot.urdf.xacro (robot description, xacro)
@@ -124,15 +124,28 @@
     </visual>
   </link>
+  <!--
+    Provisional X3 Pro location. The scan plane is 0.35 m above the ground:
+    base_link is 0.096 m above the ground, so laser_link z is 0.254 m.
+    Final drilling waits for the sampling payload and GNSS antenna layout.
+  -->
   <joint name="laser_joint" type="fixed">
-    <parent link="mast_link"/>
+    <parent link="base_link"/>
     <child link="laser_link"/>
-    <origin xyz="0 0 0.27"/>
+    <origin xyz="0.10 0 0.254" rpy="0 0 0"/>
   </joint>
   <link name="laser_link">
     <visual>
-      <geometry>
-        <cylinder radius="0.055" length="0.065"/>
+      <origin xyz="0 0 -0.021"/>
+      <geometry>
+        <box size="0.095 0.0689 0.0405"/>
       </geometry>
       <material name="blue"/>
+    </visual>
+    <visual>
+      <origin xyz="0 0 -0.005"/>
+      <geometry>
+        <cylinder radius="0.026" length="0.015"/>
+      </geometry>
+      <material name="dark"/>
     </visual>
   </link>
@@ -190,17 +203,17 @@
       <always_on>true</always_on>
       <visualize>false</visualize>
-      <update_rate>10</update_rate>
+      <update_rate>5</update_rate>
       <ray>
         <scan>
           <horizontal>
-            <samples>720</samples>
+            <samples>600</samples>
             <resolution>1</resolution>
-            <min_angle>-2.35619</min_angle>
-            <max_angle>2.35619</max_angle>
+            <min_angle>-${pi}</min_angle>
+            <max_angle>${pi}</max_angle>
           </horizontal>
         </scan>
         <range>
-          <min>0.10</min>
-          <max>20.0</max>
+          <min>0.12</min>
+          <max>8.0</max>
           <resolution>0.01</resolution>
         </range>
